Commit message: feat: integrate RPLidar A1 and configure TF tree with base_link
- Add bringup.launch.py with static TF publisher (base_link → laser_frame)
- Update amr_robot.urdf.xacro to include RPLidar A1 laser link and joint
- Update gazebo_control.xacro to reflect new sensor configuration
- Update amr_bringup package.xml with sllidar_ros2 dependency

LIDAR scan data now visualizes correctly in RViz2 with base_link as the
fixed frame. TF tree is stable: odom → base_footprint → base_link → laser_frame.

Co-Authored-By: Claude Sonnet 4.6 <noreply@anthropic.com>

File: ros2_ws/src/amr_description/urdf/amr_robot.urdf.xacro (robot description, xacro)
@@ -195,5 +195,5 @@
        Joint Z = base_height/2 + lidar_height/2 → cylinder bottom flush with chassis top.
        ===================================================================== -->
-  <link name="lidar_link">
+  <link name="laser">
     <visual>
       <origin xyz="0 0 0" rpy="0 0 0"/>
@@ -220,5 +220,5 @@
   <joint name="lidar_joint" type="fixed">
     <parent link="base_link"/>
-    <child  link="lidar_link"/>
+    <child  link="laser"/>
     <origin xyz="0.25 0 ${base_height / 2.0 + lidar_height / 2.0}" rpy="0 0 0"/>
   </joint>

File: ros2_ws/src/amr_description/urdf/gazebo_control.xacro (robot description, xacro)
@@ -17,5 +17,5 @@
     <material>Gazebo/Grey</material>
   </gazebo>
-  <gazebo reference="lidar_link">
+  <gazebo reference="laser">
     <material>Gazebo/Blue</material>
   </gazebo>

Commit message: Update AMR URDF and Gazebo control, clean up old SLAM launch files
Co-Authored-By: Claude Sonnet 4.6 <noreply@anthropic.com>

File: ros2_ws/src/amr_description/urdf/amr_robot.urdf.xacro (robot description, xacro)
@@ -3,12 +3,12 @@
   <xacro:include filename="$(find amr_description)/urdf/gazebo_control.xacro"/>
   <!-- =====================================================================
-       Locked dimensions — sourced from CLAUDE.md. Do NOT change these.
-       ===================================================================== -->
-  <xacro:property name="base_length"    value="0.600"/>   <!-- X, front-back -->
-  <xacro:property name="base_width"     value="0.500"/>   <!-- Y, side-side  -->
-  <xacro:property name="base_height"    value="0.300"/>   <!-- Z             -->
+       Physical hardware dimensions — SLLIDAR C1 + 130 mm drive wheels
+       ===================================================================== -->
+  <xacro:property name="base_length"    value="0.640"/>   <!-- X, front-back -->
+  <xacro:property name="base_width"     value="0.540"/>   <!-- Y, side-side  -->
+  <xacro:property name="base_height"    value="0.320"/>   <!-- Z             -->
   <xacro:property name="wheel_radius"   value="0.065"/>
   <xacro:property name="wheel_width"    value="0.040"/>
-  <xacro:property name="wheel_y"        value="0.275"/>   <!-- |Y| from centre -->
+  <xacro:property name="wheel_y"        value="0.270"/>   <!-- |Y| from centre = base_width/2 → 540 mm separation -->
   <xacro:property name="wheel_x"        value="-0.100"/>  <!-- rear-biased axle position -->
   <xacro:property name="caster_radius"  value="0.025"/>
@@ -17,5 +17,5 @@
   <xacro:property name="lift_width"    value="0.400"/>   <!-- Y -->
   <xacro:property name="lift_height"   value="0.020"/>   <!-- Z (thin plate) -->
-  <!-- RPLIDAR C1 — cylinder approximation -->
+  <!-- SLLIDAR C1 — cylinder approximation -->
   <xacro:property name="lidar_radius"  value="0.050"/>
   <xacro:property name="lidar_height"  value="0.060"/>
@@ -116,5 +116,5 @@
   </joint>
   <!-- =====================================================================
-       base_link — chassis box (500 × 600 × 300 mm)
+       base_link — chassis box (640 × 540 × 320 mm)
        ===================================================================== -->
   <link name="base_link">
@@ -132,11 +132,11 @@
       </geometry>
     </collision>
-    <!-- m=15 kg  box: Ixx=m/12*(w²+h²)  Iyy=m/12*(l²+h²)  Izz=m/12*(l²+w²) -->
+    <!-- m=15 kg  box 0.640×0.540×0.320: Ixx=m/12*(w²+h²)  Iyy=m/12*(l²+h²)  Izz=m/12*(l²+w²) -->
     <inertial>
       <origin xyz="0 0 0" rpy="0 0 0"/>
       <mass value="15.0"/>
-      <inertia ixx="0.425000" ixy="0" ixz="0"
-                               iyy="0.562500" iyz="0"
-                                               izz="0.762500"/>
+      <inertia ixx="0.492500" ixy="0" ixz="0"
+                               iyy="0.640000" iyz="0"
+                                               izz="0.876500"/>
     </inertial>
   </link>
@@ -148,14 +148,16 @@
   <!-- =====================================================================
        Passive casters at the four chassis corners
-       X: ±240 mm inset from ends   Y: ±180 mm inset from sides
-       ===================================================================== -->
-  <xacro:caster name="front_left"  x_pos=" 0.240" y_pos=" 0.180"/>
-  <xacro:caster name="front_right" x_pos=" 0.240" y_pos="-0.180"/>
-  <xacro:caster name="rear_left"   x_pos="-0.240" y_pos=" 0.180"/>
-  <xacro:caster name="rear_right"  x_pos="-0.240" y_pos="-0.180"/>
+       X: ±260 mm from centre (60 mm inset from ±320 mm ends)
+       Y: ±200 mm from centre (70 mm inset from ±270 mm sides)
+       ===================================================================== -->
+  <xacro:caster name="front_left"  x_pos=" 0.260" y_pos=" 0.200"/>
+  <xacro:caster name="front_right" x_pos=" 0.260" y_pos="-0.200"/>
+  <xacro:caster name="rear_left"   x_pos="-0.260" y_pos=" 0.200"/>
+  <xacro:caster name="rear_right"  x_pos="-0.260" y_pos="-0.200"/>
   <!-- =====================================================================
        Scissor-lift platform
        lift_joint origin places the platform flush on top of base_link at q=0:
-         Z = base_height/2 + lift_height/2 = 0.150 + 0.010 = 0.160 m
+         X = 0.0 m (centred on chassis for balanced weight distribution)
+         Z = base_height/2 + lift_height/2 = 0.160 + 0.010 = 0.170 m
        Prismatic displacement adds along +Z, max stroke 0.5 m.
        ===================================================================== -->
@@ -186,14 +188,15 @@
     <parent link="base_link"/>
     <child  link="lift_link"/>
-    <origin xyz="0 0 ${base_height / 2.0 + lift_height / 2.0}" rpy="0 0 0"/>
+    <origin xyz="0.0 0 ${base_height / 2.0 + lift_height / 2.0}" rpy="0 0 0"/>
     <axis xyz="0 0 1"/>
     <limit lower="0.0" upper="0.5" effort="100" velocity="0.1"/>
   </joint>
   <!-- =====================================================================
-       RPLIDAR C1  (topic: /scan)
-       Sits on top of the chassis, forward of centre.
-       Joint Z = base_height/2 + lidar_height/2 → cylinder bottom flush with chassis top.
-       ===================================================================== -->
-  <link name="laser">
+       SLLIDAR C1  (topic: /scan, frame: laser_frame)
+       Front of the top surface: X = +0.25 m from base_link centre.
+       Joint Z = base_height/2 + lidar_height/2 → cylinder bottom flush with chassis top
+       (= 0.160 + 0.030 = 0.190 m above base_link centre with 320 mm chassis height).
+       ===================================================================== -->
+  <link name="laser_frame">
     <visual>
       <origin xyz="0 0 0" rpy="0 0 0"/>
@@ -218,13 +221,13 @@
     </inertial>
   </link>
-  <joint name="lidar_joint" type="fixed">
+  <joint name="laser_joint" type="fixed">
     <parent link="base_link"/>
-    <child  link="laser"/>
-    <origin xyz="0.25 0 ${base_height / 2.0 + lidar_height / 2.0}" rpy="0 0 0"/>
+    <child  link="laser_frame"/>
+    <origin xyz="0.25 0.0 ${base_height / 2.0 + lidar_height / 2.0}" rpy="0 0 0"/>
   </joint>
   <!-- =====================================================================
        Orbbec Astra Pro depth camera  (topic: /camera/depth/points)
        Mounted on the front face of base_link, centred on the chassis height,
-       facing forward (+X). Origin X = 0.3 m = front edge of base_link.
+       facing forward (+X). Origin X = 0.32 m = front edge of base_link.
        ===================================================================== -->
   <link name="camera_link">
@@ -254,5 +257,5 @@
     <parent link="base_link"/>
     <child  link="camera_link"/>
-    <origin xyz="0.3 0 0" rpy="0 0 0"/>
+    <origin xyz="0.32 0 0" rpy="0 0 0"/>
   </joint>
 </robot>

File: ros2_ws/src/amr_description/urdf/gazebo_control.xacro (robot description, xacro)
@@ -17,5 +17,5 @@
     <material>Gazebo/Grey</material>
   </gazebo>
-  <gazebo reference="laser">
+  <gazebo reference="laser_frame">
     <material>Gazebo/Blue</material>
   </gazebo>
@@ -51,5 +51,6 @@
        Differential drive plugin
        Subscribes to /cmd_vel, publishes /odom and /tf (odom → base_footprint).
-       Wheel separation and diameter must match CLAUDE.md locked values.
+       wheel_separation = 2 * wheel_y = 2 * 0.270 = 0.540 m
+       wheel_diameter   = 2 * wheel_radius = 2 * 0.065 = 0.130 m
        ===================================================================== -->
   <gazebo>
@@ -61,6 +62,5 @@
       <left_joint>left_wheel_joint</left_joint>
       <right_joint>right_wheel_joint</right_joint>
-      <!-- LOCKED — from CLAUDE.md -->
-      <wheel_separation>0.550</wheel_separation>
+      <wheel_separation>0.540</wheel_separation>
       <wheel_diameter>0.130</wheel_diameter>
       <max_wheel_torque>200</max_wheel_torque>
